File: PCB/HackClubPCB.kicad_sch (KiCad schematic)
At the start: 22 parts, among them SW1 RotaryEncoder_Switch, SW2 SW_Push_45deg, SW3 SW_Push_45deg, SW4 SW_Push_45deg, SW5 SW_Push_45deg, SW6 SW_Push_45deg, SW7 SW_Push_45deg, SW8 SW_Push_45deg, U1 XIAO-RP2040-DIP

Commit message: pcb and cad
Parts:
- Brd1: footprint (none) -> KiCad-SSD1306-0.91-OLED-4pin-128x32:SSD1306-0.91-OLED-4pin-128x32
- SW1: footprint (none) -> Rotary_Encoder:RotaryEncoder_Alps_EC11E-Switch_Vertical_H20mm
- SW2, SW3, SW4, SW5, SW6, SW7, SW8: footprint (none) -> Button_Switch_Keyboard:SW_Cherry_MX_1.00u_PCB
Changed lines of the file:
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@@
 			)
 		)
-		(property "Footprint" ""
+		(property "Footprint" "Rotary_Encoder:RotaryEncoder_Alps_EC11E-Switch_Vertical_H20mm"
 			(at 231.394 110.49 0)
 			(effects
@@
 			)
 		)
-		(property "Footprint" ""
+		(property "Footprint" "Button_Switch_Keyboard:SW_Cherry_MX_1.00u_PCB"
 			(at 38.1 71.12 0)
 			(effects
@@
 			)
 		)
-		(property "Footprint" ""
+		(property "Footprint" "Button_Switch_Keyboard:SW_Cherry_MX_1.00u_PCB"
 			(at 101.6 44.45 0)
 			(effects
@@
 			)
 		)
-		(property "Footprint" ""
+		(property "Footprint" "Button_Switch_Keyboard:SW_Cherry_MX_1.00u_PCB"
 			(at 101.6 71.12 0)
 			(effects
@@
 			)
 		)
-		(property "Footprint" ""
+		(property "Footprint" "Button_Switch_Keyboard:SW_Cherry_MX_1.00u_PCB"
 			(at 38.1 44.45 0)
 			(effects
@@
 			)
 		)
-		(property "Footprint" ""
+		(property "Footprint" "Button_Switch_Keyboard:SW_Cherry_MX_1.00u_PCB"
 			(at 69.85 44.45 0)
 			(effects
@@
 			)
 		)
-		(property "Footprint" ""
+		(property "Footprint" "Button_Switch_Keyboard:SW_Cherry_MX_1.00u_PCB"
 			(at 133.35 44.45 0)
 			(effects
@@
 			)
 		)
-		(property "Footprint" ""
+		(property "Footprint" "KiCad-SSD1306-0.91-OLED-4pin-128x32:SSD1306-0.91-OLED-4pin-128x32"
 			(at 184.15 95.25 0)
 			(effects
@@
 			)
 		)
-		(property "Footprint" ""
+		(property "Footprint" "Button_Switch_Keyboard:SW_Cherry_MX_1.00u_PCB"
 			(at 69.85 71.12 0)
 			(effects

Commit message: fixed geeked stuff
Parts:
- U1: footprint Module:MOUDLE14P-XIAO-DIP-SMD -> Seeed Studio XIAO Series Library:XIAO-RP2040-DIP
Connections:
- net +5V: now also U1.14 (VBUS)
- net at U1.5 (GPIO6/SDA): now also Brd1.4 (SDA); no longer Brd1.3 (SCL)
- net at U1.6 (GPIO7/SCL): now also Brd1.3 (SCL); no longer Brd1.4 (SDA)
- net +3.3V: no longer names the net of U1.12 (3V3)
Other:
- moved on the sheet: Brd1
Changed lines of the file:
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@@
+	(wire
+		(pts
+			(xy 195.58 106.68) (xy 195.58 88.9)
+		)
+		(stroke
+			(width 0)
+			(type default)
+		)
+	)
 	(wire
 		(pts
@@
 	(wire
 		(pts
+			(xy 193.04 106.68) (xy 193.04 92.71)
+		)
+		(stroke
+			(width 0)
+			(type default)
+		)
+	)
+	(wire
+		(pts
 			(xy 31.75 33.02) (xy 31.75 41.91)
 		)
@@
 	(wire
 		(pts
+			(xy 195.58 88.9) (xy 209.55 88.9)
+		)
+		(stroke
+			(width 0)
+			(type default)
+		)
+	)
+	(wire
+		(pts
 			(xy 63.5 68.58) (xy 67.31 68.58)
 		)
@@
 	(wire
 		(pts
-			(xy 185.42 88.9) (xy 209.55 88.9)
-		)
-		(stroke
-			(width 0)
-			(type default)
-		)
-	)
-	(wire
-		(pts
 			(xy 232.41 43.18) (xy 257.81 43.18)
 		)
@@
 	(wire
 		(pts
-			(xy 187.96 92.71) (xy 209.55 92.71)
-		)
-		(stroke
-			(width 0)
-			(type default)
-		)
-	)
-	(wire
-		(pts
 			(xy 181.61 27.94) (xy 207.01 27.94)
 		)
@@
 	(wire
 		(pts
+			(xy 193.04 92.71) (xy 209.55 92.71)
+		)
+		(stroke
+			(width 0)
+			(type default)
+		)
+	)
+	(wire
+		(pts
 			(xy 35.56 68.58) (xy 31.75 68.58)
 		)
@@
 		(pts
 			(xy 31.75 41.91) (xy 35.56 41.91)
-		)
-		(stroke
-			(width 0)
-			(type default)
-		)
-	)
-	(wire
-		(pts
-			(xy 185.42 92.71) (xy 185.42 88.9)
 		)
 		(stroke
@@
 	)
 	(symbol
-		(lib_id "power:+3.3V")
-		(at 245.11 81.28 270)
+		(lib_id "power:+5V")
+		(at 245.11 73.66 270)
 		(unit 1)
 		(exclude_from_sim no)
@@
 		(fields_autoplaced yes)
 		(property "Reference" "#PWR01"
-			(at 241.3 81.28 0)
-			(effects
-				(font
-					(size 1.27 1.27)
-				)
-				(hide yes)
-			)
-		)
-		(property "Value" "+3.3V"
-			(at 248.92 81.2799 90)
+			(at 241.3 73.66 0)
+			(effects
+				(font
+					(size 1.27 1.27)
+				)
+				(hide yes)
+			)
+		)
+		(property "Value" "+5V"
+			(at 248.92 73.6599 90)
 			(effects
 				(font
@@
 		)
 		(property "Footprint" ""
-			(at 245.11 81.28 0)
+			(at 245.11 73.66 0)
 			(effects
 				(font
@@
 		)
 		(property "Datasheet" ""
-			(at 245.11 81.28 0)
-			(effects
-				(font
-					(size 1.27 1.27)
-				)
-				(hide yes)
-			)
-		)
-		(property "Description" "Power symbol creates a global label with name \"+3.3V\""
-			(at 245.11 81.28 0)
+			(at 245.11 73.66 0)
+			(effects
+				(font
+					(size 1.27 1.27)
+				)
+				(hide yes)
+			)
+		)
+		(property "Description" "Power symbol creates a global label with name \"+5V\""
+			(at 245.11 73.66 0)
 			(effects
 				(font
@@
 			)
 		)
-		(property "Footprint" "Module:MOUDLE14P-XIAO-DIP-SMD"
+		(property "Footprint" "Seeed Studio XIAO Series Library:XIAO-RP2040-DIP"
 			(at 227.838 100.838 0)
 			(effects
@@
 	(symbol
 		(lib_id "power:GND")
-		(at 180.34 92.71 180)
+		(at 187.96 106.68 180)
 		(unit 1)
 		(exclude_from_sim no)
@@
 		(fields_autoplaced yes)
 		(property "Reference" "#PWR02"
-			(at 180.34 86.36 0)
+			(at 187.96 100.33 0)
 			(effects
 				(font
@@
 		)
 		(property "Value" "GND"
-			(at 180.34 87.63 0)
+			(at 187.96 101.6 0)
 			(effects
 				(font
@@
 		)
 		(property "Footprint" ""
-			(at 180.34 92.71 0)
+			(at 187.96 106.68 0)
 			(effects
 				(font
@@
 		)
 		(property "Datasheet" ""
-			(at 180.34 92.71 0)
+			(at 187.96 106.68 0)
 			(effects
 				(font
@@
 		)
 		(property "Description" "Power symbol creates a global label with name \"GND\" , ground"
-			(at 180.34 92.71 0)
+			(at 187.96 106.68 0)
 			(effects
 				(font
@@
 	(symbol
 		(lib_id "power:+5V")
-		(at 182.88 92.71 0)
+		(at 190.5 106.68 0)
 		(unit 1)
 		(exclude_from_sim no)
@@
 		(fields_autoplaced yes)
 		(property "Reference" "#PWR04"
-			(at 182.88 96.52 0)
+			(at 190.5 110.49 0)
 			(effects
 				(font
@@
 		)
 		(property "Value" "+5V"
-			(at 182.88 87.63 0)
+			(at 190.5 101.6 0)
 			(effects
 				(font
@@
 		)
 		(property "Footprint" ""
-			(at 182.88 92.71 0)
+			(at 190.5 106.68 0)
 			(effects
 				(font
@@
 		)
 		(property "Datasheet" ""
-			(at 182.88 92.71 0)
+			(at 190.5 106.68 0)
 			(effects
 				(font
@@
 		)
 		(property "Description" "Power symbol creates a global label with name \"+5V\""
-			(at 182.88 92.71 0)
+			(at 190.5 106.68 0)
 			(effects
 				(font
@@
 	(symbol
 		(lib_id "SSD1306-128x64_OLED:SSD1306")
-		(at 184.15 101.6 0)
+		(at 191.77 115.57 0)
 		(unit 1)
 		(exclude_from_sim no)
@@
 		(fields_autoplaced yes)
 		(property "Reference" "Brd1"
-			(at 191.77 100.3299 0)
+			(at 199.39 114.2999 0)
 			(effects
 				(font
@@
 		)
 		(property "Value" "SSD1306"
-			(at 191.77 102.8699 0)
+			(at 199.39 116.8399 0)
 			(effects
 				(font
@@
 		)
 		(property "Footprint" "KiCad-SSD1306-0.91-OLED-4pin-128x32:SSD1306-0.91-OLED-4pin-128x32"
-			(at 184.15 95.25 0)
+			(at 191.77 109.22 0)
 			(effects
 				(font
@@
 		)
 		(property "Datasheet" ""
-			(at 184.15 95.25 0)
+			(at 191.77 109.22 0)
 			(effects
 				(font
@@
 		)
 		(property "Description" "SSD1306 OLED"
-			(at 184.15 101.6 0)
-			(effects
-				(font
+			(at 191.77 115.57 0)
+			(effects
+				(font
