File: PCB/HackClubPCB.kicad_pcb (KiCad board)
At the start: 2 copper layers, 81 x 83.3 mm, 22 parts, among them SW1 RotaryEncoder_Switch, SW2 SW_Push_45deg, SW3 SW_Push_45deg, SW4 SW_Push_45deg, SW5 SW_Push_45deg, SW6 SW_Push_45deg, SW7 SW_Push_45deg, SW8 SW_Push_45deg, U1 XIAO-RP2040-DIP

Commit message: pcb and cad
Routing:
- net Net-(U1-GPIO1/RX): track 94.7 -> 84.8 mm
- net COL1: track 110.1 -> 102.7 mm
- net GND: track 176.7 -> 174.0 mm
Other:
- board text added: "chaos's hackpad"
- board text removed: "Chaos's Hackpad"

Commit message: fixed geeked stuff
Parts:
- Brd1: footprint Display:Adafruit_SSD1306 -> KiCad-SSD1306-0.91-OLED-4pin-128x32:SSD1306-0.91-OLED-4pin-128x32
- SW1: footprint Rotary_Encoder:RotaryEncoder_Alps_EC11E-Switch_Vertical_H20mm_CircularMountingHoles -> Rotary_Encoder:RotaryEncoder_Alps_EC11E-Switch_Vertical_H20mm
- U1: footprint OPL Library:XIAO-RP2040-DIP -> Seeed Studio XIAO Series Library:XIAO-RP2040-DIP
- moved Brd1 22.6 mm to (206.1, 82.2)
- moved U1 16.8 mm to (194.7, 84.5)
Connections:
- U1 pad 12: +3.3V -> unconnected-(U1-3V3-Pad12)
- U1 pad 14: unconnected-(U1-VBUS-Pad14) -> +5V
- U1 pad 5: Net-(Brd1-SCL) -> Net-(Brd1-SDA)
- U1 pad 6: Net-(Brd1-SDA) -> Net-(Brd1-SCL)
Routing:
- net Net-(Brd1-SDA): track 40.0 -> 63.4 mm
- net +5V: track 140.9 -> 162.2 mm, vias 4 -> 2
- net Net-(Brd1-SCL): track 36.4 -> 57.2 mm
- net COL2: track 82.5 -> 64.9 mm
- net ROW1: track 139.8 -> 122.8 mm
- net COL0: track 55.8 -> 39.5 mm
- net NEOIN: track 72.1 -> 58.8 mm, vias 0 -> 1
- net GND: track 174.0 -> 161.5 mm, vias 4 -> 1
- net Net-(U1-GPIO0/TX): track 104.0 -> 91.9 mm
- net Net-(U1-GPIO1/RX): track 84.8 -> 74.2 mm
- net COL1: track 102.7 -> 92.4 mm
- net ROW0: track 125.5 -> 118.4 mm, vias 0 -> 1
- net Net-(D1-DOUT): track 27.1 -> 23.5 mm, vias 2 -> 0
- net Net-(D3-DOUT): track 26.8 -> 23.9 mm, vias 2 -> 0
- net Net-(D6-A): track 35.2 -> 33.2 mm
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Other:
- board size 81 x 83.3 mm -> 81 x 66.5 mm

Commit message: finished
Parts:
- moved D2 22.9 mm to (213.7, 114.3)
- moved D3 22.9 mm to (232.7, 114.3)
- moved D4 22.9 mm to (252.4, 114.3)
- moved D1 22.9 mm to (195.3, 114.3)
Routing:
- net NEOIN: track 58.8 -> 30.0 mm
- net +5V: track 162.2 -> 142.4 mm, vias 2 -> 1
- net COL3: track 132.7 -> 116.7 mm
- net GND: track 161.5 -> 147.1 mm
- net ROW0: track 118.4 -> 109.1 mm
- net COL1: track 92.4 -> 84.0 mm
- net Net-(D3-DOUT): track 23.9 -> 29.8 mm
- net Net-(U1-GPIO1/RX): track 74.2 -> 68.3 mm
- net Net-(U1-GPIO0/TX): track 91.9 -> 86.4 mm
- net Net-(D2-DOUT): track 23.3 -> 27.2 mm, vias 0 -> 2
- net Net-(D1-DOUT): track 23.5 -> 26.8 mm
- net Net-(D6-A): track 33.2 -> 35.2 mm
- net ROTENCS2: track 88.3 -> 89.8 mm, vias 0 -> 1
- net Net-(Brd1-SDA): track 63.4 -> 62.0 mm
- net Net-(D5-A): track 17.4 -> 16.4 mm
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Other:
- board size 81 x 66.5 mm -> 81 x 61.7 mm
