File: PCB/ChaosHackpad.kicad_pcb (KiCad board)
At the start: 2 copper layers, 81 x 61.7 mm, 22 parts, among them SW1 RotaryEncoder_Switch, SW2 SW_Push_45deg, SW3 SW_Push_45deg, SW4 SW_Push_45deg, SW5 SW_Push_45deg, SW6 SW_Push_45deg, SW7 SW_Push_45deg, SW8 SW_Push_45deg, U1 XIAO-RP2040-DIP

Commit message: added 3d models
Parts:
- SW2, SW3, SW4, SW5, SW6, SW7, SW8: footprint Button_Switch_Keyboard:SW_Cherry_MX_1.00u_PCB -> CustomSwitches:SW_Cherry_MX_1.00u_PCB
Changed lines of the file:
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@@
 		(property ki_fp_filters "D*DO?35*")
 		(sheetname "/")
-		(sheetfile "HackClubPCB.kicad_sch")
+		(sheetfile "ChaosHackpad.kicad_sch")
 		(attr through_hole)
 		(fp_line
@@
 		(property ki_fp_filters "D*DO?35*")
 		(sheetname "/")
-		(sheetfile "HackClubPCB.kicad_sch")
+		(sheetfile "ChaosHackpad.kicad_sch")
 		(attr through_hole)
 		(fp_line
@@
 		(property ki_fp_filters "D*DO?35*")
 		(sheetname "/")
-		(sheetfile "HackClubPCB.kicad_sch")
+		(sheetfile "ChaosHackpad.kicad_sch")
 		(attr through_hole)
 		(fp_line
@@
 		)
 	)
-	(footprint "Button_Switch_Keyboard:SW_Cherry_MX_1.00u_PCB"
+	(footprint "CustomSwitches:SW_Cherry_MX_1.00u_PCB"
 		(layer "F.Cu")
 		(at 235.9025 118.745)
@@
 		)
 		(sheetname "/")
-		(sheetfile "HackClubPCB.kicad_sch")
+		(sheetfile "ChaosHackpad.kicad_sch")
 		(attr through_hole)
 		(fp_line
@@
 			)
 		)
+		(model "C:/Users/joshf/Documents/Code/HackClubPCB/ChaosHackpad/Resources/Models/MX.STEP"
+			(offset
+				(xyz 4.75 2.25 5.5)
+			)
+			(scale
+				(xyz 1 1 1)
+			)
+			(rotate
+				(xyz -90 -0 -180)
+			)
+		)
 	)
 	(footprint "Diode_THT:D_DO-35_SOD27_P7.62mm_Horizontal"
@@
 		(property ki_fp_filters "D*DO?35*")
 		(sheetname "/")
-		(sheetfile "HackClubPCB.kicad_sch")
+		(sheetfile "ChaosHackpad.kicad_sch")
 		(attr through_hole)
 		(fp_line
@@
 		(property ki_fp_filters "D*DO?35*")
 		(sheetname "/")
-		(sheetfile "HackClubPCB.kicad_sch")
+		(sheetfile "ChaosHackpad.kicad_sch")
 		(attr through_hole)
 		(fp_line
@@
 		(property ki_fp_filters "LED*SK6812MINI*PLCC*3.5x3.5mm*P1.75mm*")
 		(sheetname "/")
-		(sheetfile "HackClubPCB.kicad_sch")
+		(sheetfile "ChaosHackpad.kicad_sch")
 		(attr smd)
 		(fp_line
@@
 		)
 	)
-	(footprint "Button_Switch_Keyboard:SW_Cherry_MX_1.00u_PCB"
+	(footprint "CustomSwitches:SW_Cherry_MX_1.00u_PCB"
 		(layer "F.Cu")
 		(at 197.8025 99.695)
@@
 		)
 		(sheetname "/")
-		(sheetfile "HackClubPCB.kicad_sch")
+		(sheetfile "ChaosHackpad.kicad_sch")
 		(attr through_hole)
 		(fp_line
@@
 			)
 		)
+		(model "C:/Users/joshf/Documents/Code/HackClubPCB/ChaosHackpad/Resources/Models/MX.STEP"
+			(offset
+				(xyz 4.75 2.25 5.5)
+			)
+			(scale
+				(xyz 1 1 1)
+			)
+			(rotate
+				(xyz -90 -0 -180)
+			)
+		)
 	)
 	(footprint "LED_SMD:LED_SK6812MINI_PLCC4_3.5x3.5mm_P1.75mm"
@@
 		(property ki_fp_filters "LED*SK6812MINI*PLCC*3.5x3.5mm*P1.75mm*")
 		(sheetname "/")
-		(sheetfile "HackClubPCB.kicad_sch")
+		(sheetfile "ChaosHackpad.kicad_sch")
 		(attr smd)
 		(fp_line
@@
 		)
 	)
-	(footprint "Button_Switch_Keyboard:SW_Cherry_MX_1.00u_PCB"
+	(footprint "CustomSwitches:SW_Cherry_MX_1.00u_PCB"
 		(layer "F.Cu")
 		(at 216.8525 118.745)
@@
 		)
 		(sheetname "/")
-		(sheetfile "HackClubPCB.kicad_sch")
+		(sheetfile "ChaosHackpad.kicad_sch")
 		(attr through_hole)
 		(fp_line
@@
 			)
 		)
+		(model "C:/Users/joshf/Documents/Code/HackClubPCB/ChaosHackpad/Resources/Models/MX.STEP"
+			(offset
+				(xyz 4.75 2.25 5.5)
+			)
+			(scale
+				(xyz 1 1 1)
+			)
+			(rotate
+				(xyz -90 -0 -180)
+			)
+		)
 	)
-	(footprint "Button_Switch_Keyboard:SW_Cherry_MX_1.00u_PCB"
+	(footprint "CustomSwitches:SW_Cherry_MX_1.00u_PCB"
 		(layer "F.Cu")
 		(at 216.8525 99.695)
@@
 		)
 		(sheetname "/")
-		(sheetfile "HackClubPCB.kicad_sch")
+		(sheetfile "ChaosHackpad.kicad_sch")
 		(attr through_hole)
 		(fp_line
@@
 			)
 		)
+		(model "C:/Users/joshf/Documents/Code/HackClubPCB/ChaosHackpad/Resources/Models/MX.STEP"
+			(offset
+				(xyz 4.75 2.25 5.5)
+			)
+			(scale
+				(xyz 1 1 1)
+			)
+			(rotate
+				(xyz -90 -0 -180)
+			)
+		)
 	)
 	(footprint "Diode_THT:D_DO-35_SOD27_P7.62mm_Horizontal"
@@
 		(property ki_fp_filters "D*DO?35*")
 		(sheetname "/")
-		(sheetfile "HackClubPCB.kicad_sch")
+		(sheetfile "ChaosHackpad.kicad_sch")
 		(attr through_hole)
 		(fp_line
@@
 		(property ki_fp_filters "LED*SK6812MINI*PLCC*3.5x3.5mm*P1.75mm*")
 		(sheetname "/")
-		(sheetfile "HackClubPCB.kicad_sch")
+		(sheetfile "ChaosHackpad.kicad_sch")
 		(attr smd)
 		(fp_line
@@
 		(property ki_fp_filters "LED*SK6812MINI*PLCC*3.5x3.5mm*P1.75mm*")
 		(sheetname "/")
-		(sheetfile "HackClubPCB.kicad_sch")
+		(sheetfile "ChaosHackpad.kicad_sch")
 		(attr smd)
 		(fp_line
@@
 		)
 	)
-	(footprint "Button_Switch_Keyboard:SW_Cherry_MX_1.00u_PCB"
+	(footprint "CustomSwitches:SW_Cherry_MX_1.00u_PCB"
 		(layer "F.Cu")
 		(at 197.8025 118.745)
@@
 		)
 		(sheetname "/")
-		(sheetfile "HackClubPCB.kicad_sch")
+		(sheetfile "ChaosHackpad.kicad_sch")
 		(attr through_hole)
 		(fp_line
@@
 			)
 		)
+		(model "C:/Users/joshf/Documents/Code/HackClubPCB/ChaosHackpad/Resources/Models/MX.STEP"
+			(offset
+				(xyz 4.75 2.25 5.5)
+			)
+			(scale
+				(xyz 1 1 1)
+			)
+			(rotate
+				(xyz -90 -0 -180)
+			)
+		)
 	)
 	(footprint "Rotary_Encoder:RotaryEncoder_Alps_EC11E-Switch_Vertical_H20mm"
@@
 		(property ki_fp_filters "RotaryEncoder*Switch*")
 		(sheetname "/")
-		(sheetfile "HackClubPCB.kicad_sch")
+		(sheetfile "ChaosHackpad.kicad_sch")
 		(attr through_hole)
 		(fp_line
@@
 		)
 	)
-	(footprint "Button_Switch_Keyboard:SW_Cherry_MX_1.00u_PCB"
+	(footprint "CustomSwitches:SW_Cherry_MX_1.00u_PCB"
 		(layer "F.Cu")
 		(at 254.9525 99.695)
@@
 		)
 		(sheetname "/")
-		(sheetfile "HackClubPCB.kicad_sch")
+		(sheetfile "ChaosHackpad.kicad_sch")
 		(attr through_hole)
 		(fp_line
@@
 			)
 		)
+		(model "C:/Users/joshf/Documents/Code/HackClubPCB/ChaosHackpad/Resources/Models/MX.STEP"
+			(offset
+				(xyz 4.75 2.25 5.5)
+			)
+			(scale
+				(xyz 1 1 1)
+			)
+			(rotate
+				(xyz -90 -0 -180)
+			)
+		)
 	)
 	(footprint "KiCad-SSD1306-0.91-OLED-4pin-128x32:SSD1306-0.91-OLED-4pin-128x32"
@@
 		(property ki_fp_filters "SSD1306-128x64_OLED:SSD1306")
 		(sheetname "/")
-		(sheetfile "HackClubPCB.kicad_sch")
+		(sheetfile "ChaosHackpad.kicad_sch")
 		(attr through_hole)
 		(fp_line
@@
 		(property ki_fp_filters "D*DO?35*")
 		(sheetname "/")
-		(sheetfile "HackClubPCB.kicad_sch")
+		(sheetfile "ChaosHackpad.kicad_sch")
 		(attr through_hole)
 		(fp_line
@@
 		)
 	)
-	(footprint "Button_Switch_Keyboard:SW_Cherry_MX_1.00u_PCB"
+	(footprint "CustomSwitches:SW_Cherry_MX_1.00u_PCB"
 		(layer "F.Cu")
 		(at 235.9025 99.695)
@@
 		)
 		(sheetname "/")
-		(sheetfile "HackClubPCB.kicad_sch")
+		(sheetfile "ChaosHackpad.kicad_sch")
 		(attr through_hole)
 		(fp_line
@@
 			)
 		)
+		(model "C:/Users/joshf/Documents/Code/HackClubPCB/ChaosHackpad/Resources/Models/MX.STEP"
+			(offset
+				(xyz 4.75 2.25 5.5)
+			)
+			(scale
+				(xyz 1 1 1)
+			)
+			(rotate
+				(xyz -90 -0 -180)
+			)
+		)
 	)
 	(footprint "Seeed Studio XIAO Series Library:XIAO-RP2040-DIP"
@@
 		)
 		(sheetname "/")
-		(sheetfile "HackClubPCB.kicad_sch")
+		(sheetfile "ChaosHackpad.kicad_sch")
 		(attr smd)
 		(fp_line
@@
 		(property ki_fp_filters "D*DO?35*")
 		(sheetname "/")
-		(sheetfile "HackClubPCB.kicad_sch")
+		(sheetfile "ChaosHackpad.kicad_sch")
 		(attr through_hole)
 		(fp_line
